File: cad/mainboard/mainboard.kicad_pcb (KiCad board)
At the start: 4 copper layers, 89.6 x 90 mm, 76 parts, among them J101 RJ45_Shielded, J102 RJ45_Shielded, J103 RJ45_Shielded, J104 RJ45_Shielded, J105 RJ45_Shielded, J106 Conn_01x02_MountingPin, J107 Conn_01x04, J108 Conn_01x04, J109 ftdi_conn, Q101 BSS138, Q102 BSS138, Q103 BSS138, Q104 BSS138, Q105 BSS138, Q106 BSS138, Q107 BSS138, Q108 BSS138, Q109 BSS138, Q110 BSS138, Q111 BSS138, Q112 BSS138, SW101 SW_Push, SW102 SW_Push, U101 XL1509, U102 ESP32-WROOM-32U, U103 AMS1117-3.3, U104 Trans_CAN_SN65HVD230DR

Commit message: add cad stuff
Routing:
- net /SCL_OUT: track 152.7 -> 156.9 mm
- net GND: vias 407 -> 406
